File: hardware/relay.sch (KiCad schematic (older format))
At the start: 13 parts, among them J1 LOAD, K1 SRD-05VDC-SL-C, Q1 PMBT3904, U5 PC817X2CSP9F, U6 CC6902SO-10A

Commit message: checkpoint commit
Parts:
- J1: footprint TerminalBlock:TerminalBlock_Altech_AK300-3_P5.00mm -> TerminalBlock_Phoenix:TerminalBlock_Phoenix_MKDS-1,5-3_1x03_P5.00mm_Horizontal
Connections:
- net at J1.2 (Pin_2), U6.3 (IP-), U6.4 (IP-): no longer K1.1
- net at U6.1 (IP+), U6.2 (IP+): now also K1.1; no longer J1.3 (Pin_3), K1.3
- new net: J1.3 (Pin_3), K1.3
Other:
- moved on the sheet: J2, U4
Changed lines of the file:
@@
 $Descr A4 11693 8268
 encoding utf-8
-Sheet 2 5
+Sheet 3 5
 Title "Relay Subsystem"
 Date "2021-06-11"
@@
 AR Path="/60CBD77D/60C3AACC" Ref="Q3"  Part="1"
 AR Path="/60CBD7BB/60C3AACC" Ref="Q4"  Part="1"
-F 0 "Q1" H 5541 4296 50  0000 L CNN
+F 0 "Q2" H 5541 4296 50  0000 L CNN
 F 1 "PMBT3904" H 5541 4205 50  0000 L CNN
 F 2 "Package_TO_SOT_SMD:SOT-23" H 5550 4350 50  0001 C CNN
@@
 AR Path="/60CBD77D/60C3DB9C" Ref="R9"  Part="1"
 AR Path="/60CBD7BB/60C3DB9C" Ref="R12"  Part="1"
-F 0 "R3" V 4800 4200 50  0000 L CNN
+F 0 "R6" V 4800 4200 50  0000 L CNN
 F 1 "1K" V 4600 4200 50  0000 L CNN
 F 2 "Resistor_SMD:R_0805_2012Metric" V 4630 4250 50  0001 C CNN
@@
 AR Path="/60CBD77D/60C3E090" Ref="R7"  Part="1"
 AR Path="/60CBD7BB/60C3E090" Ref="R10"  Part="1"
-F 0 "R1" V 3000 4000 50  0000 L CNN
+F 0 "R4" V 3000 4000 50  0000 L CNN
 F 1 "200R" V 2800 3950 50  0000 L CNN
 F 2 "Resistor_SMD:R_0805_2012Metric" V 2830 4050 50  0001 C CNN
@@
 L Connector:Screw_Terminal_01x03 J1
 U 1 1 60C4BBD2
-P 5850 2350
+P 6600 2350
 AR Path="/60C36AE5/60C4BBD2" Ref="J1"  Part="1"
 AR Path="/60CBD6BF/60C4BBD2" Ref="J2"  Part="1"
 AR Path="/60CBD77D/60C4BBD2" Ref="J3"  Part="1"
 AR Path="/60CBD7BB/60C4BBD2" Ref="J4"  Part="1"
-F 0 "J1" V 5900 2050 50  0000 L CNN
-F 1 "LOAD" V 5800 1950 50  0000 L CNN
-F 2 "TerminalBlock:TerminalBlock_Altech_AK300-3_P5.00mm" H 5850 2350 50  0001 C CNN
-F 3 "~" H 5850 2350 50  0001 C CNN
-	1    5850 2350
-	0    -1   -1   0
+F 0 "J2" H 6550 2050 50  0000 L CNN
+F 1 "LOAD" H 6550 2150 50  0000 L CNN
+F 2 "TerminalBlock_Phoenix:TerminalBlock_Phoenix_MKDS-1,5-3_1x03_P5.00mm_Horizontal" H 6600 2350 50  0001 C CNN
+F 3 "~" H 6600 2350 50  0001 C CNN
+	1    6600 2350
+	1    0    0    1
 $EndComp
 Wire Wire Line
@@
 AR Path="/60CBD77D/60C544FE" Ref="D6"  Part="1"
 AR Path="/60CBD7BB/60C544FE" Ref="D8"  Part="1"
-F 0 "D2" V 4604 3530 50  0000 L CNN
+F 0 "D4" V 4604 3530 50  0000 L CNN
 F 1 "1N4007F" V 4695 3530 50  0000 L CNN
 F 2 "Diode_SMD:D_SMA" H 4650 3450 50  0001 C CNN
@@
 AR Path="/60CBD77D/60C3D896" Ref="R8"  Part="1"
 AR Path="/60CBD7BB/60C3D896" Ref="R11"  Part="1"
-F 0 "R2" H 4370 3196 50  0000 L CNN
+F 0 "R5" H 4370 3196 50  0000 L CNN
 F 1 "200R" H 4370 3105 50  0000 L CNN
 F 2 "Resistor_SMD:R_0805_2012Metric" V 4230 3150 50  0001 C CNN
@@
 AR Path="/60CBD77D/60C370D4" Ref="K3"  Part="1"
 AR Path="/60CBD7BB/60C370D4" Ref="K4"  Part="1"
-F 0 "K1" H 5350 3900 50  0000 C CNN
+F 0 "K2" H 5350 3900 50  0000 C CNN
 F 1 "SRD-05VDC-SL-C" H 5050 3800 50  0000 C CNN
 F 2 "Relay_THT:Relay_SPDT_SANYOU_SRD_Series_Form_C" H 6100 3400 50  0001 L CNN
@@
 AR Path="/60CBD77D/60C91E1E" Ref="#PWR06"  Part="1"
 AR Path="/60CBD7BB/60C91E1E" Ref="#PWR08"  Part="1"
-F 0 "#PWR01" H 5450 4600 50  0001 C CNN
+F 0 "#PWR08" H 5450 4600 50  0001 C CNN
 F 1 "GND" H 5455 4677 50  0000 C CNN
 F 2 "" H 5450 4850 50  0001 C CNN
@@
 	4300 2650 4300 2850
 Wire Wire Line
-	5750 2550 5750 3150
-Wire Wire Line
-	5850 2550 5850 2700
-Wire Wire Line
-	5850 2700 6250 2700
-Wire Wire Line
-	6250 3750 5850 3750
-Wire Wire Line
-	6250 2700 6250 3550
-Wire Wire Line
-	5950 2550 5950 3050
-Wire Wire Line
-	5450 4650 7150 4650
-Wire Wire Line
-	7150 3550 7150 4650
-Wire Wire Line
-	6450 3050 5950 3050
-Connection ~ 5950 3050
-Wire Wire Line
-	5950 3050 5950 3150
-Wire Wire Line
-	6450 3450 6450 3550
-Wire Wire Line
-	6450 3550 6250 3550
-Connection ~ 6250 3550
-Wire Wire Line
-	6250 3550 6250 3750
-Wire Wire Line
-	6450 3050 6450 3250
+	5450 4650 7000 4650
+Wire Wire Line
+	7000 3550 7000 4650
 $Comp
 L CustomComponents:PC817X2CSP9F U5
@@
 AR Path="/60CBD6BF/60D16537" Ref="U3"  Part="1"
 AR Path="/60CBD7BB/60D16537" Ref="U7"  Part="1"
-F 0 "U1" H 3600 4475 50  0000 C CNN
+F 0 "U3" H 3600 4475 50  0000 C CNN
 F 1 "PC817X2CSP9F" H 3600 4384 50  0000 C CNN
 F 2 "CustomComponents:PC817X2CSP9F" H 3400 3950 50  0001 L CIN
@@
 L CustomComponents:CC690XSO-XA U6
 U 1 1 60D16B35
-P 6800 3400
+P 6650 3400
 AR Path="/60CBD77D/60D16B35" Ref="U6"  Part="1"
 AR Path="/60C36AE5/60D16B35" Ref="U2"  Part="1"
 AR Path="/60CBD6BF/60D16B35" Ref="U4"  Part="1"
 AR Path="/60CBD7BB/60D16B35" Ref="U8"  Part="1"
-F 0 "U2" H 6800 3815 50  0000 C CNN
-F 1 "CC6902SO-10A" H 6800 3724 50  0000 C CNN
-F 2 "CustomComponents:CC690XSO-XA" H 6800 3100 50  0001 C CNN
-F 3 "" H 6800 3600 50  0001 C CNN
-	1    6800 3400
-	1    0    0    -1
-$EndComp
-Connection ~ 6450 3550
-Wire Wire Line
-	6450 3250 6450 3350
-Connection ~ 6450 3250
-Wire Wire Line
-	5450 2850 7200 2850
-Wire Wire Line
-	7150 3250 7200 3250
-Wire Wire Line
-	7200 2850 7200 3250
+F 0 "U4" H 6650 3815 50  0000 C CNN
+F 1 "CC6902SO-10A" H 6650 3724 50  0000 C CNN
+F 2 "CustomComponents:CC690XSO-XA" H 6650 3100 50  0001 C CNN
+F 3 "" H 6650 3600 50  0001 C CNN
+	1    6650 3400
+	1    0    0    -1
+$EndComp
+Wire Wire Line
+	5450 2850 7050 2850
+Wire Wire Line
+	7000 3250 7050 3250
+Wire Wire Line
+	7050 2850 7050 3250
 $Comp
 L Device:LED D1
@@
 AR Path="/60CBD77D/60C3C98C" Ref="D5"  Part="1"
 AR Path="/60CBD7BB/60C3C98C" Ref="D7"  Part="1"
-F 0 "D1" V 4300 3750 50  0000 C CNN
+F 0 "D3" V 4300 3750 50  0000 C CNN
 F 1 "LED" V 4200 3750 50  0000 C CNN
 F 2 "LED_SMD:LED_0805_2012Metric" H 4300 3600 50  0001 C CNN
@@
 AR Path="/60CBD77D/60CD3C14" Ref="#PWR019"  Part="1"
 AR Path="/60CBD7BB/60CD3C14" Ref="#PWR020"  Part="1"
-F 0 "#PWR017" H 4300 2500 50  0001 C CNN
+F 0 "#PWR020" H 4300 2500 50  0001 C CNN
 F 1 "+5V" H 4315 2823 50  0000 C CNN
 F 2 "" H 4300 2650 50  0001 C CNN
@@
 AR Path="/60CBD77D/60C94FE5" Ref="C5"  Part="1"
 AR Path="/60CBD7BB/60C94FE5" Ref="C7"  Part="1"
-F 0 "C1" H 7865 3946 50  0000 L CNN
+F 0 "C3" H 7865 3946 50  0000 L CNN
 F 1 "100P" H 7865 3855 50  0000 L CNN
 F 2 "Capacitor_SMD:C_0805_2012Metric" H 7788 3750 50  0001 C CNN
@@
 AR Path="/60CBD77D/60CDBA1D" Ref="R15"  Part="1"
 AR Path="/60CBD7BB/60CDBA1D" Ref="R16"  Part="1"
-F 0 "R13" V 7293 3350 50  0000 C CNN
+F 0 "R14" V 7293 3350 50  0000 C CNN
 F 1 "100R" V 7384 3350 50  0000 C CNN
 F 2 "Resistor_SMD:R_0805_2012Metric" V 7430 3350 50  0001 C CNN
@@
 AR Path="/60CBD77D/60C99EC6" Ref="C6"  Part="1"
 AR Path="/60CBD7BB/60C99EC6" Ref="C8"  Part="1"
-F 0 "C2" H 8415 3946 50  0000 L CNN
+F 0 "C4" H 8415 3946 50  0000 L CNN
 F 1 "100N" H 8415 3855 50  0000 L CNN
 F 2 "Capacitor_SMD:C_0805_2012Metric" H 8338 3750 50  0001 C CNN
@@
 	1    0    0    -1
 $EndComp
-Connection ~ 7150 4650
-Wire Wire Line
-	7150 4650 7750 4650
 Wire Wire Line
 	7650 3350 7750 3350
-Wire Wire Line
-	7150 3350 7350 3350
 Wire Wire Line
 	8300 4050 8300 4650
@@
 Wire Wire Line
 	7750 4650 8300 4650
-Connection ~ 7200 2850
-Wire Wire Line
-	7200 2850 8300 2850
 Connection ~ 7750 3350
 Wire Wire Line
@@
 Text Notes 5550 4500 0    50   ~ 0
 0.4A max (0.2A limit) \nat hFE = 100
+Connection ~ 7000 4650
+Connection ~ 7050 2850
+Wire Wire Line
+	7000 4650 7750 4650
+Wire Wire Line
+	7050 2850 8300 2850
+Wire Wire Line
+	7000 3350 7350 3350
+Wire Wire Line
+	5750 3150 5750 2450
+Wire Wire Line
+	5950 2250 6400 2250
+Wire Wire Line
+	5950 2250 5950 3150
+Wire Wire Line
+	6400 2450 5750 2450
+Wire Wire Line
+	6300 3250 6300 3300
+Wire Wire Line
+	6300 3450 6300 3500
+Wire Wire Line
+	5850 3750 6100 3750
+Wire Wire Line
+	6100 3750 6100 3300
+Wire Wire Line
+	6100 3300 6300 3300
+Connection ~ 6300 3300
+Wire Wire Line
+	6300 3300 6300 3350
+Wire Wire Line
+	6300 3500 6200 3500
+Wire Wire Line
+	6200 3500 6200 2350
+Wire Wire Line
+	6200 2350 6400 2350
+Connection ~ 6300 3500
+Wire Wire Line
+	6300 3500 6300 3550
 $EndSCHEMATC
