File: hardware/power-extender.kicad_pcb (KiCad board)
At the start: 2 copper layers, 90 x 71 mm, 78 parts, among them J1 IFACE RPI, J11 LOAD, J2 IFACE PASS, J21 LOAD, J3 AUX ANALOG, J31 LOAD, J4 AUX DIGITAL, J41 LOAD, K11 SRD-05VDC-SL-C, K21 SRD-05VDC-SL-C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

Commit message: save file
Other:
- rule trace_min: 0.15 -> 0.21

Commit message: Add rev 1.1 fabrication files
Parts:
- J1, J2, J3, J4: footprint Connector_JST:JST_XH_B5B-XH-A_1x05_P2.50mm_Vertical -> CustomComponents:JST_XH_B5B-XH-A_1x05_P2.54mm_Vertical
Routing:
- net +5V: track 304.4 -> 305.7 mm
Other:
- board text added: "Power Extender REV1.1 CHRZ 2021"
- board text removed: "Power Extender REV1 CHRZ 2021"
