File: hardware/relay-mir.sch (KiCad schematic (older format))
At the start: 13 parts, among them J11 LOAD, K11 SRD-05VDC-SL-C, Q11 PMBT3904, U31 PC817X2CSP9F, U32 CC6902SO-10A

Commit message: relay layout checkpoint
Connections:
- net at U32.1 (IP+), U32.2 (IP+): now also J11.2 (Pin_2); no longer K11.1
- net at U32.3 (IP-), U32.4 (IP-): now also K11.1; no longer J11.2 (Pin_2)
Changed lines of the file:
@@
 Wire Wire Line
 	6400 2450 5750 2450
-Wire Wire Line
-	6300 3250 6300 3300
-Wire Wire Line
-	6300 3450 6300 3500
 $Comp
 L Device:R R12
@@
 $EndComp
 Wire Wire Line
-	5850 3750 6100 3750
+	6300 3250 6300 3350
 Wire Wire Line
-	6100 3750 6100 3300
+	6300 3450 6300 3550
 Wire Wire Line
-	6100 3300 6300 3300
-Connection ~ 6300 3300
+	6300 3750 6300 3550
 Wire Wire Line
-	6300 3300 6300 3350
+	5850 3750 6300 3750
+Connection ~ 6300 3550
 Wire Wire Line
-	6300 3500 6200 3500
+	6300 3250 6300 2350
+Connection ~ 6300 3250
 Wire Wire Line
-	6200 3500 6200 2350
-Wire Wire Line
-	6200 2350 6400 2350
-Connection ~ 6300 3500
-Wire Wire Line
-	6300 3500 6300 3550
+	6300 2350 6400 2350
 $EndSCHEMATC

Commit message: Add bjt pulldown, prepare for export
Parts:
- added R25: 10K, Resistor_SMD:R_0805_2012Metric, symbol Device:R
- C11: Description / Value (none) -> CAP CER 100PF MAX. 5% MIN. 10V 0805 SMD; Distributor (none) -> Any; Distributor part # (none) -> TBD; Manufacturer (none) -> TBD; Manufacturer Part # (none) -> TBD; Package / Footprint (none) -> 0805; Type (none) -> SMD
- C12: Description / Value (none) -> CAP CER 100NF MAX. 5% MIN. 10V 0805 SMD; Distributor (none) -> Any; Distributor part # (none) -> TBD; Manufacturer (none) -> TBD; Manufacturer Part # (none) -> TBD; Package / Footprint (none) -> 0805; Type (none) -> SMD
- D11: Description / Value (none) -> LED RED 2V 0805 SMD; Distributor (none) -> LCSC; Distributor part # (none) -> C72037; Manufacturer (none) -> Everlight Elec; Manufacturer Part # (none) -> 17-21SURC/S530-A3/TR8; Package / Footprint (none) -> 0805; Type (none) -> SMD
- D12: Description / Value (none) -> DIODE 1N4007 SMAF; Distributor (none) -> LCSC; Distributor part # (none) -> C110856; Manufacturer (none) -> Shikues; Manufacturer Part # (none) -> 1N4007F; Package / Footprint (none) -> SMAF; Type (none) -> SMD
- J11: Description / Value (none) -> CONN SCREW TERMINAL PITCH-5.0MM 3 PIN 20A; Distributor (none) -> LCSC; Distributor part # (none) -> C8270; Manufacturer (none) -> Ningbo Kangnex Elec; Manufacturer Part # (none) -> WJ128V-5.0-3P; Package / Footprint (none) -> Through-Hole; Type (none) -> THT
- K11: Description / Value (none) -> RELAY 5V 10A; Distributor (none) -> LCSC; Distributor part # (none) -> C35449; Manufacturer (none) -> Ningbo Songle Relay; Manufacturer Part # (none) -> SRD-05VDC-SL-C; Package / Footprint (none) -> Through-Hole; Type (none) -> THT
- Q11: Description / Value (none) -> BJT NPN SOT-23-3; Distributor (none) -> LCSC; Distributor part # (none) -> C8667; Manufacturer (none) -> Nexperia; Manufacturer Part # (none) -> PMBT3904,215; Package / Footprint (none) -> SOT-23-3; Type (none) -> SMD
- R11, R12: Description / Value (none) -> RES 200 OHM MAX. 1% MIN. 1/8W 0805 SMD; Distributor (none) -> Any; Distributor part # (none) -> TBD; Manufacturer (none) -> TBD; Manufacturer Part # (none) -> TBD; Package / Footprint (none) -> 0805; Type (none) -> SMD
- R13: Description / Value (none) -> RES 1K OHM MAX. 1% MIN. 1/8W 0805 SMD; Distributor (none) -> Any; Distributor part # (none) -> TBD; Manufacturer (none) -> TBD; Manufacturer Part # (none) -> TBD; Package / Footprint (none) -> 0805; Type (none) -> SMD
- R14: Description / Value (none) -> RES 100 OHM MAX. 1% MIN. 1/8W 0805 SMD; Distributor (none) -> Any; Distributor part # (none) -> TBD; Manufacturer (none) -> TBD; Manufacturer Part # (none) -> TBD; Package / Footprint (none) -> 0805; Type (none) -> SMD
- U31: Description / Value (none) -> IC OPTOCOUPLER SMD-4; Distributor (none) -> LCSC; Distributor part # (none) -> C66405; Manufacturer (none) -> Sharp Microelectronics; Manufacturer Part # (none) -> PC817X2CSP9F; Package / Footprint (none) -> SMD-4; Type (none) -> SMD
- U32: Description / Value (none) -> IC CURRENT SENSOR 5V 10A SOP-8; Distributor (none) -> LCSC; Distributor part # (none) -> C350865; Manufacturer (none) -> Cross Chip; Manufacturer Part # (none) -> CC6902SO-10A; Package / Footprint (none) -> SOP-8; Type (none) -> SMD
Connections:
- net GND: now also R25.2
- net at R13.1, U31.3: now also R25.1
Other:
- note added: "0.2A at hFE = 50"
- note removed: "0.4A max (0.2A limit) \nat hFE = 100"

Commit message: rev1 final touchups
Parts:
- D12: footprint Diode_SMD:D_SMA -> CustomComponents:D_SMAF
Changed lines of the file:
@@
 $Descr A4 11693 8268
 encoding utf-8
-Sheet 4 5
+Sheet 5 5
 Title "Relay Subsystem"
 Date "2021-06-11"
@@
 AR Path="/60CBD77D/60C91E1E" Ref="#PWR032"  Part="1"
 AR Path="/60CBD7BB/60C91E1E" Ref="#PWR042"  Part="1"
-F 0 "#PWR042" H 5450 4600 50  0001 C CNN
+F 0 "#PWR022" H 5450 4600 50  0001 C CNN
 F 1 "GND" H 5455 4677 50  0000 C CNN
 F 2 "" H 5450 4850 50  0001 C CNN
@@
 AR Path="/60CBD77D/60D1BED6" Ref="#PWR031"  Part="1"
 AR Path="/60CBD7BB/60D1BED6" Ref="#PWR041"  Part="1"
-F 0 "#PWR041" H 4300 2500 50  0001 C CNN
+F 0 "#PWR021" H 4300 2500 50  0001 C CNN
 F 1 "+5V" H 4315 2823 50  0000 C CNN
 F 2 "" H 4300 2650 50  0001 C CNN
@@
 F 0 "D22" V 4604 3530 50  0000 L CNN
 F 1 "1N4007F" V 4695 3530 50  0000 L CNN
-F 2 "Diode_SMD:D_SMA" H 4650 3450 50  0001 C CNN
+F 2 "CustomComponents:D_SMAF" H 4650 3450 50  0001 C CNN
 F 3 "~" H 4650 3450 50  0001 C CNN
 F 4 "DIODE 1N4007 SMAF" H 4650 3450 50  0001 C CNN "Description / Value"

Commit message: Add rev 1.1 fabrication files
Changed lines of the file:
@@
 $Descr A4 11693 8268
 encoding utf-8
-Sheet 5 5
+Sheet 4 5
 Title "Relay Subsystem"
 Date "2021-06-11"
@@
 AR Path="/60CBD77D/60D1BECC" Ref="Q31"  Part="1"
 AR Path="/60CBD7BB/60D1BECC" Ref="Q41"  Part="1"
-F 0 "Q21" H 5541 4296 50  0000 L CNN
+F 0 "Q41" H 5541 4296 50  0000 L CNN
 F 1 "PMBT3904" H 5541 4205 50  0000 L CNN
 F 2 "Package_TO_SOT_SMD:SOT-23" H 5550 4350 50  0001 C CNN
@@
 AR Path="/60CBD77D/60C3DB9C" Ref="R33"  Part="1"
 AR Path="/60CBD7BB/60C3DB9C" Ref="R43"  Part="1"
-F 0 "R23" V 4800 4200 50  0000 L CNN
+F 0 "R43" V 4800 4200 50  0000 L CNN
 F 1 "1K" V 4600 4200 50  0000 L CNN
 F 2 "Resistor_SMD:R_0805_2012Metric" V 4630 4250 50  0001 C CNN
@@
 AR Path="/60CBD77D/60D1BED1" Ref="J31"  Part="1"
 AR Path="/60CBD7BB/60D1BED1" Ref="J41"  Part="1"
-F 0 "J21" H 6550 2050 50  0000 L CNN
+F 0 "J41" H 6550 2050 50  0000 L CNN
 F 1 "LOAD" H 6550 2150 50  0000 L CNN
 F 2 "TerminalBlock_Phoenix:TerminalBlock_Phoenix_MKDS-1,5-3_1x03_P5.00mm_Horizontal" H 6600 2350 50  0001 C CNN
@@
 AR Path="/60CBD77D/60C370D4" Ref="K31"  Part="1"
 AR Path="/60CBD7BB/60C370D4" Ref="K41"  Part="1"
-F 0 "K21" H 5350 3900 50  0000 C CNN
+F 0 "K41" H 5350 3900 50  0000 C CNN
 F 1 "SRD-05VDC-SL-C" H 5050 3800 50  0000 C CNN
 F 2 "Relay_THT:Relay_SPDT_SANYOU_SRD_Series_Form_C" H 6100 3400 50  0001 L CNN
@@
 AR Path="/60CBD77D/60C91E1E" Ref="#PWR032"  Part="1"
 AR Path="/60CBD7BB/60C91E1E" Ref="#PWR042"  Part="1"
-F 0 "#PWR022" H 5450 4600 50  0001 C CNN
+F 0 "#PWR042" H 5450 4600 50  0001 C CNN
 F 1 "GND" H 5455 4677 50  0000 C CNN
 F 2 "" H 5450 4850 50  0001 C CNN
@@
 AR Path="/60CBD6BF/60D16B35" Ref="U22"  Part="1"
 AR Path="/60CBD7BB/60D16B35" Ref="U42"  Part="1"
-F 0 "U22" H 6650 3815 50  0000 C CNN
+F 0 "U42" H 6650 3815 50  0000 C CNN
 F 1 "CC6902SO-10A" H 6650 3724 50  0000 C CNN
 F 2 "CustomComponents:CC690XSO-XA" H 6650 3100 50  0001 C CNN
@@
 AR Path="/60CBD77D/60D1BED6" Ref="#PWR031"  Part="1"
 AR Path="/60CBD7BB/60D1BED6" Ref="#PWR041"  Part="1"
-F 0 "#PWR021" H 4300 2500 50  0001 C CNN
+F 0 "#PWR041" H 4300 2500 50  0001 C CNN
 F 1 "+5V" H 4315 2823 50  0000 C CNN
 F 2 "" H 4300 2650 50  0001 C CNN
@@
 AR Path="/60CBD77D/60C94FE5" Ref="C31"  Part="1"
 AR Path="/60CBD7BB/60C94FE5" Ref="C41"  Part="1"
-F 0 "C21" H 7865 3946 50  0000 L CNN
+F 0 "C41" H 7865 3946 50  0000 L CNN
 F 1 "100P" H 7865 3855 50  0000 L CNN
 F 2 "Capacitor_SMD:C_0805_2012Metric" H 7788 3750 50  0001 C CNN
@@
 AR Path="/60CBD77D/60CDBA1D" Ref="R34"  Part="1"
 AR Path="/60CBD7BB/60CDBA1D" Ref="R44"  Part="1"
-F 0 "R24" V 7293 3350 50  0000 C CNN
+F 0 "R44" V 7293 3350 50  0000 C CNN
 F 1 "100R" V 7384 3350 50  0000 C CNN
 F 2 "Resistor_SMD:R_0805_2012Metric" V 7430 3350 50  0001 C CNN
@@
 AR Path="/60CBD77D/60C99EC6" Ref="C32"  Part="1"
 AR Path="/60CBD7BB/60C99EC6" Ref="C42"  Part="1"
-F 0 "C22" H 8415 3946 50  0000 L CNN
+F 0 "C42" H 8415 3946 50  0000 L CNN
 F 1 "100N" H 8415 3855 50  0000 L CNN
 F 2 "Capacitor_SMD:C_0805_2012Metric" H 8338 3750 50  0001 C CNN
@@
 AR Path="/60CBD77D/60D1BECE" Ref="R32"  Part="1"
 AR Path="/60CBD7BB/60D1BECE" Ref="R42"  Part="1"
-F 0 "R22" H 4370 3196 50  0000 L CNN
+F 0 "R42" H 4370 3196 50  0000 L CNN
 F 1 "200R" H 4370 3105 50  0000 L CNN
 F 2 "Resistor_SMD:R_0805_2012Metric" V 4230 3150 50  0001 C CNN
@@
 AR Path="/60CBD77D/60D1BED2" Ref="D32"  Part="1"
 AR Path="/60CBD7BB/60D1BED2" Ref="D42"  Part="1"
-F 0 "D22" V 4604 3530 50  0000 L CNN
+F 0 "D42" V 4604 3530 50  0000 L CNN
 F 1 "1N4007F" V 4695 3530 50  0000 L CNN
 F 2 "CustomComponents:D_SMAF" H 4650 3450 50  0001 C CNN
@@
 AR Path="/60CBD77D/60D1BECD" Ref="D31"  Part="1"
 AR Path="/60CBD7BB/60D1BECD" Ref="D41"  Part="1"
-F 0 "D21" V 4300 3750 50  0000 C CNN
+F 0 "D41" V 4300 3750 50  0000 C CNN
 F 1 "LED" V 4200 3750 50  0000 C CNN
 F 2 "LED_SMD:LED_0805_2012Metric" H 4300 3600 50  0001 C CNN
@@
 AR Path="/60CBD6BF/60D1BED8" Ref="U21"  Part="1"
 AR Path="/60CBD7BB/60D1BED8" Ref="U41"  Part="1"
-F 0 "U21" H 3600 4475 50  0000 C CNN
+F 0 "U41" H 3600 4475 50  0000 C CNN
 F 1 "PC817X2CSP9F" H 3600 4384 50  0000 C CNN
 F 2 "CustomComponents:PC817X2CSP9F" H 3400 3950 50  0001 L CIN
@@
 AR Path="/60CBD77D/60D1BED0" Ref="R31"  Part="1"
 AR Path="/60CBD7BB/60D1BED0" Ref="R41"  Part="1"
-F 0 "R21" V 3000 4000 50  0000 L CNN
+F 0 "R41" V 3000 4000 50  0000 L CNN
 F 1 "200R" V 2800 3950 50  0000 L CNN
 F 2 "Resistor_SMD:R_0805_2012Metric" V 2830 4050 50  0001 C CNN
@@
 AR Path="/60CBD6BF/60D7FFE4" Ref="R25"  Part="1"
 AR Path="/60CBD7BB/60D7FFE4" Ref="R45"  Part="1"
-F 0 "R25" H 4270 4446 50  0000 L CNN
+F 0 "R45" H 4270 4446 50  0000 L CNN
 F 1 "10K" H 4270 4355 50  0000 L CNN
 F 2 "Resistor_SMD:R_0805_2012Metric" V 4130 4400 50  0001 C CNN
